File: OneInchEye.kicad_sch (KiCad schematic)
At the start: 84 parts, among them J1 FH12A-22S-0.5SH(55), J2 QWIIC_CONNECTORJS-1MM, Q1 DMG2302UK-7, Q2 DMG2302UK-7, U1 LP5907MFX-1.8, U2 LP5907MFX-2.9, U3 IMX283EQJC, U4 TMP117MAIDRVR, U5 ECS-2520MV-240-DN-TR, U6 AP3418KTR-G1

Commit message: Update to v1.4
Parts:
- removed Q1, Q2: DMG2302UK-7, Package_TO_SOT_SMD:SOT-23, symbol Transistor_FET:DMN30H4D0L
- added C39, C40, C41: 100nF, Capacitor_SMD:C_0402_1005Metric, symbol Device:C
- added FB4: BLM18KG102SN1D, Inductor_SMD:L_0402_1005Metric, symbol Device:FerriteBead
- added JP1: Jumper_3_Open, Jumper:SolderJumper-3_P1.3mm_Open_RoundedPad1.0x1.5mm_NumberLabels, symbol Jumper:Jumper_3_Open
- added JP2: SolderJumper_2_Open, Jumper:SolderJumper-2_P1.3mm_Open_RoundedPad1.0x1.5mm, symbol Jumper:SolderJumper_2_Open
- added R9: 10K, Resistor_SMD:R_0402_1005Metric, symbol Device:R
- added U7: TCA9406DC, footprints:TCA9406DCUR, symbol Interface:TCA9406DC
- added U8: ATECC608A-MAHDA, Package_DFN_QFN:DFN-8-1EP_3x2mm_P0.5mm_EP1.3x1.5mm, symbol Security:ATECC608A-MAHDA
- U4: value TMP117MAIDRVR -> TMP117AIDRVR
Connections:
- net +1V8: now also C39.1, U7.3 (VCCA), U7.6 (OE); no longer C35.2, U4.5 (V+)
- net +3V3: now also C40.1, C41.1, FB4.1, JP1.3 (B), U7.7 (VCCB), U8.8 (VCC)
- net CAM_EN: now also JP2.2 (B), R9.1; no longer J1.6 (Pin_6)
- net GND: now also C39.2, C40.2, C41.2, JP1.1 (A), U7.2 (GND), U8.4 (GND), U8.9 (EP)
- net SCL_1V8: now also U7.4 (SDA_A); no longer U4.1 (SCL)
- net SCL_3V3: now also U4.1 (SCL), U7.1 (SDA_B), U8.6 (SCL)
- net SDA_1V8: now also U7.5 (SCL_A); no longer U4.6 (SDA)
- net SDA_3V3: now also U4.6 (SDA), U7.8 (SCL_B), U8.5 (SDA)
- new net: JP1.2 (C), R9.2
- new net: C35.2, FB4.2, U4.5 (V+)
- new net: J1.6 (Pin_6), JP2.1 (A)
Other:
- moved on the sheet: C35

Commit message: Adding IMU and update board outline to 39mm square
Parts:
- removed J1: FH12A-22S-0.5SH(55), Connector_FFC-FPC:Hirose_FH12-22S-0.5SH_1x22-1MP_P0.50mm_Horizontal, symbol Connector:Conn_01x22_Female
- removed J2: QWIIC_CONNECTORJS-1MM, Connector_JST:JST_SH_SM04B-SRSS-TB_1x04-1MP_P1.00mm_Horizontal, symbol SparkFun-Connectors:QWIIC_CONNECTORJS-1MM
- removed TP11, TP2, TP3, TP9: TestPoint, TestPoint:TestPoint_Pad_D1.0mm, symbol Connector:TestPoint
- added C42: 100n, Capacitor_SMD:C_0402_1005Metric, symbol Device:C
- added C43: 10nF, Capacitor_SMD:C_0402_1005Metric, symbol Device:C
- added C44: 2.2uF, Capacitor_SMD:C_0402_1005Metric, symbol Device:C
- added J1: Conn_01x22_Shielded, footprints:TF3822S05SV830, symbol Connector_Generic_Shielded:Conn_01x22_Shielded
- added J2: Conn_01x04_Shielded, Connector_JST:JST_SH_BM04B-SRSS-TB_1x04-1MP_P1.00mm_Vertical, symbol Connector_Generic_Shielded:Conn_01x04_Shielded
- added J3, J4: Conn_Coaxial, U.FL_Hirose_U.FL-R-SMT-1_Vertical, symbol Connector:Conn_Coaxial
- added JPR1, JPR2: 0R, Resistor_SMD:R_0402_1005Metric, symbol Device:R
- added U9: ICM-42688-P, footprints:PQFN50P300X250X97-14N, symbol ICM-42688-P:ICM-42688-P
- FL1, FL2, FL3, FL4, FL5: value DLP11SN900HL2L -> KCZ1210AH900HRTD25
- R2, R3: value 10K -> DNP
- U5: value ECS-2520MV-240-DN-TR -> ECS-2520S18-240-FN-TR
Connections:
- net +1V8: now also C42.1, C43.1, C44.1, U9.12 (AP_CS), U9.5 (VDDIO), U9.8 (VDD)
- net +3V3: now also J1.1 (Pin_1), J2.2 (Pin_2)
- net CAM_EN: now also JPR2.1
- net GND: now also C42.2, C43.2, C44.2, J1.10 (Pin_10), J1.13 (Pin_13), J1.16 (Pin_16), J1.19 (Pin_19), J1.22 (Pin_22), J1.4 (Pin_4), J1.7 (Pin_7), J1.MP (Shield), J2.1 (Pin_1), J2.MP (Shield), J3.2 (Ext), J4.2 (Ext), JPR1.2, U9.1 (AP_SDO/AP_AD0), U9.10 (RESV_10), U9.11 (RESV_11), U9.2 (RESV_2), U9.3 (RESV_3), U9.6 (GND), U9.7 (RESV_7)
- net SCL_1V8: now also U9.13 (AP_SCL/AP_SCLK)
- net SCL_3V3: now also J1.3 (Pin_3), J2.4 (Pin_4)
- net SDA_1V8: now also U9.14 (AP_SDA/AP_SDIO/AP_SDI)
- net SDA_3V3: now also J1.2 (Pin_2), J2.3 (Pin_3)
- net XHS: now also J4.1 (In)
- net XVS: now also J3.1 (In), U9.9 (INT2/FSYNC/CLKIN)
- net D3_N: now reaches FL5.2
- net D3_N: now also J1.9 (Pin_9)
- net D3_P: now reaches FL5.3
- net D3_P: now also J1.8 (Pin_8)
- net D1_N: now reaches FL2.2
- net D1_N: now also J1.18 (Pin_18)
- net D1_P: now reaches FL2.3
- net D1_P: now also J1.17 (Pin_17)
- net at JP1.2 (C), R9.2: now also JPR1.1
- net D0_N: now reaches FL1.2
- net D0_N: now also J1.21 (Pin_21)
- net D0_P: now reaches FL1.3
- net D0_P: now also J1.20 (Pin_20)
- net CLK_N: now reaches FL3.2
- net CLK_N: now also J1.15 (Pin_15)
- net CLK_P: now reaches FL3.3
- net CLK_P: now also J1.14 (Pin_14)
- net D2_N: now reaches FL4.2
- net D2_N: now also J1.12 (Pin_12)
- net D2_P: now reaches FL4.3
- net D2_P: now also J1.11 (Pin_11)
- net at JP2.1 (A): now also J1.6 (Pin_6), JPR2.2
Other:
- note added: "HCMOS 24Mhz 1.8V"
- note added: "I2C ADDR: 0x60"
- note added: "I2C ADDR: 0x68"
- moved on the sheet: C1, C10, C11, C12, C13, C14, C15, C16, C17, C18, C19, C2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

Commit message: V2.1
Parts:
- removed C26: 4.7uF, Capacitor_SMD:C_0603_1608Metric, symbol Device:C
- removed C41: 100nF, Capacitor_SMD:C_0402_1005Metric, symbol Device:C
- removed JP1: Jumper_3_Open, Jumper:SolderJumper-3_P1.3mm_Open_RoundedPad1.0x1.5mm_NumberLabels, symbol Jumper:Jumper_3_Open
- removed JP2: SolderJumper_2_Open, Jumper:SolderJumper-2_P1.3mm_Open_RoundedPad1.0x1.5mm, symbol Jumper:SolderJumper_2_Open
- removed JPR1, JPR2: 0R, Resistor_SMD:R_0402_1005Metric, symbol Device:R
- removed TP10: TestPoint, TestPoint:TestPoint_Pad_D1.0mm, symbol Connector:TestPoint
- removed U2: LP5907MFX-2.9, Package_TO_SOT_SMD:SOT-23-5, symbol Regulator_Linear:LP5907MFX-2.9
- removed U8: ATECC608A-MAHDA, Package_DFN_QFN:DFN-8-1EP_3x2mm_P0.5mm_EP1.3x1.5mm, symbol Security:ATECC608A-MAHDA
- added C26: NFM18CC101R1C3D, footprints:NFM18CC101R1C3D, symbol Device:C_Feedthrough
- added C45: 1uF, Capacitor_SMD:C_0402_1005Metric, symbol Device:C
- added C46: 10nF, Capacitor_SMD:C_0402_1005Metric, symbol Device:C
- added C47: 10uF, Capacitor_SMD:C_0603_1608Metric, symbol Device:C
- added R10: 3.01K, Resistor_SMD:R_0402_1005Metric, symbol Device:R
- added R11: 1.15K, Resistor_SMD:R_0402_1005Metric, symbol Device:R
- added U2: TPS7A90, Package_DFN_QFN:Texas_S-PDSO-N10_EP1.2x2mm, symbol Regulator_Linear:TPS7A90
- C34: value 4.7uF -> 10uF
- C42: value 100n -> 100nF
- FB4: value BLM18KG102SN1D -> BLM15PX800SN1D
- U9: footprint footprints:PQFN50P300X250X97-14N -> footprints:IIM42352
Connections:
- net +2V9: now also C46.2, C47.1, R10.2, U2.1 (OUT), U2.2 (OUT); no longer C34.1
- net CAM_EN: now also J1.6 (Pin_6), U2.7 (EN)
- net GND: now also R9.2, C26.2, C45.2, C47.2, R11.1, U2.11 (GND), U2.4 (GND)
- net at FB2.2: now also C26.1
- new net: C26.3, C34.1, U2.10 (IN), U2.6 (SS_CTRL), U2.9 (IN)
- new net: C46.1, R10.1, R11.2, U2.3 (FB)
- new net: C45.1, U2.8 (NR/SS)
Other:
- note removed: "I2C ADDR: 0x60"
- moved on the sheet: C25, C33, C35, FB1, FB2, FB4, TP12, TP13, TP14, TP8, U1, U4
